File: Projects/26-27 Induction Tachometer/Tachometer/Tachometer.kicad_sch (KiCad schematic)
At the start: 33 parts, among them J1 DTF13-6P, Q1 NPN, U1 TJA1050DRG, U2 MCP2515-I, U3 LM311, U4 NE555P, X1 ${ALTIUM_VALUE}

Commit message: Set up for Workshop
Parts:
- removed VR1: 3362P-1-103, Potentiometer_THT:Potentiometer_ACP_CA9-V10_Vertical, symbol 0_3362P-1-103:3362P-1-103
- added R12: 1K, Resistor_THT:R_Axial_DIN0207_L6.3mm_D2.5mm_P10.16mm_Horizontal, symbol Device:R_US
- added RV1: R_Potentiometer, Potentiometer_THT:Potentiometer_Bourns_3296W_Vertical, symbol Device:R_Potentiometer
- C2, C3, C4, C5: DATASHEET * -> (none)
- D1, U5: value ~ -> (none)
- R1, R10, R11, R13, R2, R3, R4, R5, R6, R7, R8, R9: footprint Resistor_THT:R_Axial_DIN0204_L3.6mm_D1.6mm_P7.62mm_Horizontal -> Resistor_THT:R_Axial_DIN0207_L6.3mm_D2.5mm_P10.16mm_Horizontal
- U1: DATASHEET https://atta.szlcsc.com/upload/public/pdf/source/20231229/9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 -> (none)
- U2: DATASHEET https://atta.szlcsc.com/upload/public/pdf/source/20221108/5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 -> (none)
Connections:
- net 555 input: now also U3.1 (GND), R12.1
- net GND: now also RV1.3; no longer U3.1 (GND), U5.2 (Inductor_Out)
- net VCC: now also R1.1, R12.2
- net at R8.2, R9.2: now also U3.2 (+)
- net at C13.1, U4.6 (THR), U4.7 (DIS): now also RV1.2; no longer R7.1
- net at U5.1 (Inductor_In): now also RV1.1; no longer R1.1
- new net: R7.1, U5.2 (Inductor_Out)
Other:
- moved on the sheet: R4, R6, R7, U5
