File: Shared Elements/CAN Module Circuit 26-27/CAN Module Circuit 26-27.kicad_sch (KiCad schematic)
At the start: 9 parts, among them U1 TJA1050DRG, U2 MCP2515-I, X1 ${ALTIUM_VALUE}

Commit message: Set up gitignore to exclude Kicad backups
Parts:
- C2, C3, C4, C5: DATASHEET * -> (none)
- U1: DATASHEET https://atta.szlcsc.com/upload/public/pdf/source/20231229/9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 -> (none)
- U2: DATASHEET https://atta.szlcsc.com/upload/public/pdf/source/20221108/5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 -> (none)

Commit message: Set up for Workshop
Parts:
- R3: footprint Resistor_THT:R_Axial_DIN0204_L3.6mm_D1.6mm_P7.62mm_Horizontal -> Resistor_THT:R_Axial_DIN0207_L6.3mm_D2.5mm_P5.08mm_Vertical
Changed lines of the file:
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@@
 	(symbol
 		(lib_id "CAN Integration-altium-import:VCC_BAR")
-		(at 149.86 106.68 180)
+		(at 149.86 106.68 90)
 		(unit 1)
 		(body_style 1)
@@
 		)
 		(property "Value" "VCC"
-			(at 149.86 102.87 0)
+			(at 153.67 106.68 0)
 			(show_name no)
 			(do_not_autoplace no)
@@
 			)
 		)
-		(property "Footprint" "Resistor_THT:R_Axial_DIN0204_L3.6mm_D1.6mm_P7.62mm_Horizontal"
+		(property "Footprint" "Resistor_THT:R_Axial_DIN0207_L6.3mm_D2.5mm_P5.08mm_Vertical"
 			(at 99.314 92.964 90)
 			(hide yes)
