File: Projects/Dash/Dashboard.kicad_pcb (KiCad board)
At the start: 2 copper layers, 4 parts, among them J1 DTF13-6P, J2 Conn_01x02_Socket, U2 Adafruit-CAN-BFF-SMD

Commit message: [2026-09-19] Dash REV 1 Done
Parts:
- added G***: LOGO, LOGO, F.Cu at (161.8, 106.9)
- added J10: R2C3 (0x75), Connector_PinHeader_2.54mm:PinHeader_1x05_P2.54mm_Vertical, F.Cu at (162.1, 91.8)
- added J11: Top Row Button, Connector_PinHeader_2.54mm:PinHeader_1x02_P2.54mm_Vertical, F.Cu at (136.6, 108.4)
- added J12: Bottom Row Button, Connector_PinHeader_2.54mm:PinHeader_1x02_P2.54mm_Vertical, F.Cu at (130.8, 108.4)
- added J3: Tach Servo Header, Connector_PinHeader_2.54mm:PinHeader_1x03_P2.54mm_Vertical, F.Cu at (116.3, 109.6)
- added J4: Speed Servo Header, Connector_PinHeader_2.54mm:PinHeader_1x03_P2.54mm_Vertical, F.Cu at (122.0, 109.6)
- added J5: R1C1 (0x70), Connector_PinHeader_2.54mm:PinHeader_1x05_P2.54mm_Vertical, F.Cu at (116.3, 82.0)
- added J6: R1C2 (0x71), Connector_PinHeader_2.54mm:PinHeader_1x05_P2.54mm_Vertical, F.Cu at (139.2, 82.0)
- added J7: R1C3 (0x72), Connector_PinHeader_2.54mm:PinHeader_1x05_P2.54mm_Vertical, F.Cu at (162.1, 82.0)
- added J8: R2C1 (0x73), Connector_PinHeader_2.54mm:PinHeader_1x05_P2.54mm_Vertical, F.Cu at (116.3, 91.8)
- added J9: R2C2 (0x74), Connector_PinHeader_2.54mm:PinHeader_1x05_P2.54mm_Vertical, F.Cu at (139.2, 91.8)
- added REF**: MountingHole_3.2mm_M3, MountingHole:MountingHole_3.2mm_M3, F.Cu at (183.6, 144.2)
- added REF**: MountingHole_3.2mm_M3, MountingHole:MountingHole_3.2mm_M3, F.Cu at (104.5, 144.2)
- added REF**: MountingHole_3.2mm_M3, MountingHole:MountingHole_3.2mm_M3, F.Cu at (183.6, 86.9)
- added REF**: MountingHole_3.2mm_M3, MountingHole:MountingHole_3.2mm_M3, F.Cu at (104.5, 86.9)
- J1: value DTF13-6P -> Deutsch Connector; moved to B.Cu
- J2: value Conn_01x02_Socket -> CAN BFF Intercepting Header; footprint Connector_PinSocket_2.54mm:PinSocket_1x02_P2.54mm_Vertical -> Connector_PinHeader_2.54mm:PinHeader_1x03_P2.54mm_Vertical
- moved J1 82.9 mm to (171.7, 57.7), turned to 0 degrees
- moved J2 77.0 mm to (153.7, 127.3), turned to 0 degrees
- moved U2 70.4 mm to (120.4, 129.9), turned to -90 degrees
- moved A1 59.7 mm to (109.7, 62.1), turned to -90 degrees
Connections:
- A1 pad D10: unconnected-(A1-PadD10) -> SERVO_TACH
- A1 pad D5: SERVO_TACH -> unconnected-(A1-PadD5)
- A1 pad D6: SERVO_SPEED -> unconnected-(A1-PadD6)
- A1 pad D7: unconnected-(A1-PadD7) -> BUTTON_TOP
- A1 pad D8: unconnected-(A1-PadD8) -> BUTTON_BOTTOM
- A1 pad D9: unconnected-(A1-PadD9) -> SERVO_SPEED
- J2 pad 1: CAN_OUTPUT_H -> CAN_OUTPUT_L
- J2 pad 2: CAN_OUTPUT_L -> CAN_OUTPUT_H
Routing:
- net +5V: track 0.00 -> 217.6 mm
- net I2C_SDA: track 0.00 -> 94.2 mm
- net I2C_SCL: track 0.00 -> 92.9 mm
- net CAN_OUTPUT_H: track 0.00 -> 90.1 mm
- net BUTTON_TOP: track 0.00 -> 82.8 mm
- net CAN_OUTPUT_L: track 0.00 -> 81.1 mm
- net BUTTON_BOTTOM: track 0.00 -> 77.7 mm
- net SERVO_SPEED: track 0.00 -> 69.0 mm
- net SERVO_TACH: track 0.00 -> 62.3 mm
- net GND: track 0.00 -> 2.93 mm, vias 0 -> 1
- added copper zone on B.Cu, net GND
Other:
- board outline added: 90 x 100 mm
- board text added: "Dashboard 2026-REV-1 Designed by Adam Esch in Tucson, Arizona"

Commit message: Guess who forgot the SPI bus 😂
Parts:
- added REF**: Fiducial_0.75mm_Mask1.5mm, Fiducial:Fiducial_0.75mm_Mask1.5mm, F.Cu at (183.6, 137.2)
- added REF**: Fiducial_0.75mm_Mask1.5mm, Fiducial:Fiducial_0.75mm_Mask1.5mm, F.Cu at (104.5, 137.2)
- added REF**: Fiducial_0.75mm_Mask1.5mm, Fiducial:Fiducial_0.75mm_Mask1.5mm, F.Cu at (104.5, 93.9)
- added REF**: Fiducial_0.75mm_Mask1.5mm, Fiducial:Fiducial_0.75mm_Mask1.5mm, F.Cu at (183.6, 93.9)
Connections:
- A1 pad D11: unconnected-(A1-D11_MOSI-PadD11) -> SPI_SI
- A1 pad D12: unconnected-(A1-D12_MISO-PadD12) -> SPI_SO
- A1 pad D13: unconnected-(A1-D13_SCK-PadD13) -> SPI_SCK
- A1 pad D5: unconnected-(A1-PadD5) -> CAN_INT
- A1 pad D6: unconnected-(A1-PadD6) -> CAN_CS
- A1 pad GND2: unconnected-(A1-GND-PadGND2) -> GND
Routing:
- net SPI_SO: track 0.00 -> 105.1 mm
- net SPI_SI: track 0.00 -> 102.9 mm
- net CAN_INT: track 0.00 -> 90.1 mm, vias 0 -> 1
- net SPI_SCK: track 0.00 -> 79.4 mm
- net CAN_CS: track 0.00 -> 77.1 mm, vias 0 -> 1
- net +5V: track 217.6 -> 200.9 mm
Other:
- outline, holes or cut-outs redrawn
