File: Projects/26-27 VR Tach EX/VR_Sensor_Tach_Cam/VR_Sensor_Tach_Cam.kicad_sch (KiCad schematic)
At the start: 17 parts, among them J1 DTF13-6P, U1 Variable Reluctance Sensor In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, U2 MCP2515-I, U3 TJA1050DRG, X1 ${ALTIUM_VALUE}

Commit message: Updated PCB with all Components and text
Parts:
- C1: footprint (none) -> Capacitor_THT:CP_Radial_D5.0mm_P2.50mm
- R1, R2, R_pullup1: footprint (none) -> Resistor_THT:R_Axial_DIN0204_L3.6mm_D1.6mm_P5.08mm_Horizontal
- R3: footprint Resistor_THT:R_Axial_DIN0207_L6.3mm_D2.5mm_P5.08mm_Vertical -> Resistor_THT:R_Axial_DIN0204_L3.6mm_D1.6mm_P5.08mm_Horizontal
- U1: footprint MAX9924UAUB_:SOP50P490X110-10N -> MAX9924UAUB_ (1):SOP50P490X110-10N
- VR Sensor1: footprint Package_SO:SOIC-28W_7.5x17.9mm_P1.27mm -> MAX9924UAUB_ (1):VR Sensor
Changed lines of the file:
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@@
 			)
 		)
-		(property "Value" "0"
+		(property "Value" "GND"
 			(at 147.32 154.94 0)
 			(hide yes)
@@
 			)
 		)
-		(property "Value" "0"
+		(property "Value" "GND"
 			(at 33.02 180.34 0)
 			(hide yes)
@@
 			)
 		)
-		(property "Footprint" "MAX9924UAUB_:SOP50P490X110-10N"
+		(property "Footprint" "MAX9924UAUB_ (1):SOP50P490X110-10N"
 			(at 85.09 69.85 0)
 			(hide yes)
@@
 			)
 		)
-		(property "Value" "0"
+		(property "Value" "GND"
 			(at 41.91 180.34 0)
 			(hide yes)
@@
 			)
 		)
-		(property "Value" "0"
+		(property "Value" "GND"
 			(at 114.3 152.4 0)
 			(hide yes)
@@
 			)
 		)
-		(property "Value" "0"
+		(property "Value" "GND"
 			(at 160.02 158.75 0)
 			(hide yes)
@@
 			)
 		)
-		(property "Footprint" ""
+		(property "Footprint" "Resistor_THT:R_Axial_DIN0204_L3.6mm_D1.6mm_P5.08mm_Horizontal"
 			(at 113.792 53.34 90)
 			(hide yes)
@@
 			)
 		)
-		(property "Footprint" "Package_SO:SOIC-28W_7.5x17.9mm_P1.27mm"
+		(property "Footprint" "MAX9924UAUB_ (1):VR Sensor"
 			(at 24.13 54.61 0)
 			(hide yes)
@@
 			)
 		)
-		(property "Footprint" ""
+		(property "Footprint" "Capacitor_THT:CP_Radial_D5.0mm_P2.50mm"
 			(at 53.0352 58.42 0)
 			(hide yes)
@@
 			)
 		)
-		(property "Value" "0"
+		(property "Value" "GND"
 			(at 107.95 179.07 0)
 			(hide yes)
@@
 			)
 		)
-		(property "Footprint" ""
+		(property "Footprint" "Resistor_THT:R_Axial_DIN0204_L3.6mm_D1.6mm_P5.08mm_Horizontal"
 			(at 43.18 51.308 90)
 			(hide yes)
@@
 			)
 		)
-		(property "Footprint" "Resistor_THT:R_Axial_DIN0207_L6.3mm_D2.5mm_P5.08mm_Vertical"
+		(property "Footprint" "Resistor_THT:R_Axial_DIN0204_L3.6mm_D1.6mm_P5.08mm_Horizontal"
 			(at 57.404 156.464 90)
 			(hide yes)
@@
 			)
 		)
-		(property "Footprint" ""
+		(property "Footprint" "Resistor_THT:R_Axial_DIN0204_L3.6mm_D1.6mm_P5.08mm_Horizontal"
 			(at 43.18 61.468 90)
 			(hide yes)
