File: Projects/26-27 VR Tach EX/VR_Sensor_Tach_Cam/VR_Sensor_Tach_Cam.kicad_pcb (KiCad board)
At the start: 2 copper layers, 50 x 50 mm, 22 parts, among them J1 DTF13-6P, U1 Variable Reluctance Sensor In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, U2 MCP2515-I, U3 TJA1050DRG, X1 8MHz

Commit message: VR Tach PCB Updated with Baja Logo
Parts:
- added G***: LOGO, Baja Logo for PCB New:Baja Logo, B.Cu at (63.0, 80.0)
Other:
- board text added: "Variable Reluctance Tachometer"

Commit message: Updated PCB
Parts:
- removed the G*** at (68.0, 62.0)
- added G***: LOGO, VR_Sensor_Tach_Cam:PHD_Image, B.Cu at (89.2, 82.0)
- moved VR Sensor 43.5 mm to (59.5, 54.5), turned to -90 degrees
- moved R2 35.1 mm to (64.9, 57.0), turned to 0 degrees
- moved R1 35.0 mm to (65.0, 52.5), turned to 0 degrees
- moved C3 28.0 mm to (81.0, 87.0)
- moved C5 28.0 mm to (74.5, 87.0)
- moved R3 27.4 mm to (46.9, 79.0)
- moved C6 27.0 mm to (81.0, 80.0)
- moved C4 27.0 mm to (74.5, 80.0)
- moved U3 22.0 mm to (49.0, 86.0)
- moved C1 21.6 mm to (74.0, 53.5), turned to -90 degrees
- moved U2 21.5 mm to (59.0, 84.0)
- moved X1 21.3 mm to (69.0, 83.8)
- moved G*** 20.4 mm to (78.8, 67.0)
- moved R_pullup1 13.6 mm to (83.0, 52.5), turned to 180 degrees
- moved C2 13.4 mm to (89.8, 62.0), turned to 0 degrees
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Routing:
- net GND: track 176.0 -> 14.6 mm, vias 0 -> 8
- net Low: track 79.0 -> 34.2 mm, vias 0 -> 2
- net +5V: track 151.3 -> 117.3 mm
- net Cout: track 42.1 -> 19.0 mm
- net SCK: track 36.0 -> 15.6 mm
- net High: track 63.2 -> 43.7 mm, vias 0 -> 2
- net CS: track 16.6 -> 21.2 mm, vias 0 -> 1
- net Net-(U1-IN-): track 12.9 -> 8.76 mm
- net SI: track 31.1 -> 27.1 mm, vias 0 -> 1
- net Net-(U2-OSC1): track 17.5 -> 14.1 mm
- net SO: track 29.7 -> 26.7 mm, vias 0 -> 1
- net Net-(U1-IN+): track 12.2 -> 9.55 mm
- net INT: track 26.0 -> 23.8 mm, vias 0 -> 1
- net Net-(U2-~{RESET}): track 7.18 -> 5.09 mm
- net Net-(U2-RXCAN): track 7.16 -> 5.59 mm
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- added copper zone on B.Cu, net GND
