File: Projects/IMU/IMU Circuit 26-27.kicad_sch (KiCad schematic)
At the start: 19 parts, among them J1 DTF Connector, U1 TJA1050DRG, U2 MCP2515-I, U3 TM171, X1 ${ALTIUM_VALUE}

Commit message: term R added
Parts:
- added R4: 120, Resistor_THT:R_Axial_DIN0207_L6.3mm_D2.5mm_P5.08mm_Vertical, symbol Device:R_US
Connections:
- net High: now also R4.2
- net Low: now also R4.1
Other:
- note added: "Termination Resistor (Optional)"
Changed lines of the file:
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@@
 		)
 	)
+	(rectangle
+		(start 175.26 100.33)
+		(end 205.74 127)
+		(stroke
+			(width 0)
+			(type dot)
+		)
+		(fill
+			(type none)
+		)
+	)
 	(text "10K"
 		(exclude_from_sim no)
@@
 		)
 	)
+	(text "Termination Resistor\n(Optional)"
+		(exclude_from_sim no)
+		(at 190.754 107.696 0)
+		(effects
+			(font
+				(size 1.778 1.778)
+				(thickness 0.3556)
+				(bold yes)
+			)
+			(justify bottom)
+		)
+	)
 	(text "22pF"
 		(exclude_from_sim no)
@@
 	(wire
 		(pts
+			(xy 190.5 120.65) (xy 190.5 123.19)
+		)
+		(stroke
+			(width 0)
+			(type default)
+		)
+	)
+	(wire
+		(pts
 			(xy 59.69 179.07) (xy 59.69 180.34)
 		)
@@
 	(wire
 		(pts
+			(xy 190.5 110.49) (xy 190.5 113.03)
+		)
+		(stroke
+			(width 0)
+			(type default)
+		)
+	)
+	(wire
+		(pts
 			(xy 168.91 114.3) (xy 160.02 114.3)
 		)
@@
 		)
 	)
+	(global_label "Low"
+		(shape input)
+		(at 190.5 123.19 180)
+		(fields_autoplaced yes)
+		(effects
+			(font
+				(size 1.27 1.27)
+			)
+			(justify right)
+		)
+		(property "Intersheetrefs" "${INTERSHEET_REFS}"
+			(at 184.0072 123.19 0)
+			(hide yes)
+			(show_name no)
+			(do_not_autoplace no)
+			(effects
+				(font
+					(size 1.27 1.27)
+				)
+				(justify right)
+			)
+		)
+	)
 	(global_label "High"
 		(shape input)
@@
 	(global_label "High"
 		(shape input)
+		(at 190.5 110.49 0)
+		(fields_autoplaced yes)
+		(effects
+			(font
+				(size 1.27 1.27)
+			)
+			(justify left)
+		)
+		(property "Intersheetrefs" "${INTERSHEET_REFS}"
+			(at 197.7185 110.49 0)
+			(hide yes)
+			(show_name no)
+			(do_not_autoplace no)
+			(effects
+				(font
+					(size 1.27 1.27)
+				)
+				(justify left)
+			)
+		)
+	)
+	(global_label "High"
+		(shape input)
 		(at 147.32 143.51 0)
 		(fields_autoplaced yes)
@@
 				)
 			)
+		)
+	)
+	(symbol
+		(lib_id "Device:R_US")
+		(at 190.5 116.84 180)
+		(unit 1)
+		(body_style 1)
+		(exclude_from_sim no)
+		(in_bom yes)
+		(on_board yes)
+		(in_pos_files yes)
+		(dnp no)
+		(fields_autoplaced yes)
+		(property "Reference" "R4"
+			(at 193.04 115.5699 0)
+			(show_name no)
+			(do_not_autoplace no)
+			(effects
+				(font
+					(size 1.27 1.27)
+				)
+				(justify right)
+			)
+		)
+		(property "Value" "120"
+			(at 193.04 118.1099 0)
+			(show_name no)
+			(do_not_autoplace no)
+			(effects
+				(font
+					(size 1.27 1.27)
+				)
+				(justify right)
+			)
+		)
+		(property "Footprint" "Resistor_THT:R_Axial_DIN0207_L6.3mm_D2.5mm_P5.08mm_Vertical"
+			(at 189.484 116.586 90)
+			(hide yes)
+			(show_name no)
+			(do_not_autoplace no)
+			(effects
+				(font
+					(size 1.27 1.27)
+				)
+			)
+		)
+		(property "Datasheet" ""
+			(at 190.5 116.84 0)
+			(hide yes)
+			(show_name no)
+			(do_not_autoplace no)
+			(effects
+				(font
+					(size 1.27 1.27)
+				)
+			)
+		)
+		(property "Description" "Resistor, US symbol"
+			(at 190.5 116.84 0)
+			(hide yes)
+			(show_name no)
+			(do_not_autoplace no)
+			(effects
+				(font
+					(size 1.27 1.27)
+				)
+			)
+		)
+		(pin "1"
+		)
+		(pin "2"
+		)
+		(instances
+			(project "IMU Circuit 26-27"
+				(path "/d185ddb1-e4c7-4aec-9e87-37dceb424272"
+					(reference "R4")
+					(unit 1)
+				)
+			)
