File: Projects/Displacement Sensor 2/Displacement Sensor 2.kicad_sch (KiCad schematic)
At the start: 10 parts, among them U1 TJA1050DRG, U2 MCP2515-I, X1 ${ALTIUM_VALUE}

Commit message: Custom symbol
Parts:
- added U3: (no value), symbol Displacement Pins:Displacement_pins
Connections:
- net at A1.19 (A0): now also U3.3 (SIGNAL)
Changed lines of the file:
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@@
-	(wire
-		(pts
-			(xy 147.32 64.77) (xy 147.32 77.47)
-		)
-		(stroke
-			(width 0)
-			(type default)
-		)
-	)
 	(wire
 		(pts
@@
 	(wire
 		(pts
+			(xy 102.87 77.47) (xy 143.51 77.47)
+		)
+		(stroke
+			(width 0)
+			(type default)
+		)
+	)
+	(wire
+		(pts
 			(xy 210.82 135.89) (xy 207.01 135.89)
 		)
@@
 	(wire
 		(pts
-			(xy 102.87 77.47) (xy 147.32 77.47)
-		)
-		(stroke
-			(width 0)
-			(type default)
-		)
-	)
-	(wire
-		(pts
 			(xy 154.94 134.62) (xy 160.02 134.62)
 		)
@@
 	(wire
 		(pts
+			(xy 143.51 77.47) (xy 143.51 62.23)
+		)
+		(stroke
+			(width 0)
+			(type default)
+		)
+	)
+	(wire
+		(pts
 			(xy 135.89 114.3) (xy 135.89 127)
+		)
+		(stroke
+			(width 0)
+			(type default)
+		)
+	)
+	(wire
+		(pts
+			(xy 143.51 62.23) (xy 152.4 62.23)
 		)
 		(stroke
@@
 					(unit 1)
 				)
+			)
+		)
+	)
+	(symbol
+		(lib_id "Displacement Pins:Displacement_pins")
+		(at 152.4 59.69 0)
+		(unit 1)
+		(body_style 1)
+		(exclude_from_sim no)
+		(in_bom yes)
+		(on_board yes)
+		(in_pos_files yes)
+		(dnp no)
+		(fields_autoplaced yes)
+		(property "Reference" "U3"
+			(at 163.83 60.9599 0)
+			(show_name no)
+			(do_not_autoplace no)
+			(effects
+				(font
+					(size 1.27 1.27)
+				)
+				(justify left)
+			)
+		)
+		(property "Value" ""
+			(at 152.4 59.69 0)
+			(show_name no)
+			(do_not_autoplace no)
+			(effects
+				(font
+					(size 1.27 1.27)
+				)
+			)
+		)
+		(property "Footprint" ""
+			(at 152.4 59.69 0)
+			(hide yes)
+			(show_name no)
+			(do_not_autoplace no)
+			(effects
+				(font
+					(size 1.27 1.27)
+				)
+			)
+		)
+		(property "Datasheet" ""
+			(at 152.4 59.69 0)
+			(hide yes)
+			(show_name no)
+			(do_not_autoplace no)
+			(effects
+				(font
+					(size 1.27 1.27)
+				)
+			)
+		)
+		(property "Description" ""
+			(at 152.4 59.69 0)
+			(hide yes)
+			(show_name no)
+			(do_not_autoplace no)
+			(effects
+				(font
+					(size 1.27 1.27)
+				)
+			)
+		)
+		(pin "4"
+		)
+		(pin "1"
+		)
+		(pin "2"
+		)
+		(pin "3"
+		)
+		(instances
+			(project "Displacement Sensor 2"
+				(path "/cef208de-ab75-42af-9ed7-91863f7f236f"
+					(reference "U3")
+					(unit 1)
+				)

Commit message: Finished displacement schem
Parts:
- added J1: DTF13-6P, DTF13-6P:TE_DTF13-6P, symbol DTF13-6P:DTF13-6P
- added unit 1 of U1
- added unit 1 of U2
- added U3: (no value), symbol Displacement Pins:Displacement_pins
- renumbered U3 to U0
Connections:
- net CS: now also A1.13 (D10)
- net High: now also J1.4, J1.5
- net INT: now also A1.5 (D2)
- net Low: now also J1.2, J1.3
- net SCK: now also A1.16 (D13)
- net SI: now also A1.14 (D11)
- net SO: now also A1.15 (D12)
- net 5V: now reaches U0.1 (5V)
- net 5V: now also A1.27 (+5V), J1.6, U1.1 (5V), U2.1 (5V), U3.1 (5V)
- net GND: now reaches U0.2 (GND)
- net GND: now also A1.29 (GND), A1.4 (GND), U0.4 (CGND), J1.1, U1.2 (GND), U1.4 (CGND), U2.2 (GND), U2.4 (CGND), U3.2 (GND), U3.4 (CGND)
- net at A1.20 (A1): now also U1.3 (SIGNAL)
- net at A1.21 (A2): now also U2.3 (SIGNAL)
- net at A1.22 (A3): now also U3.3 (SIGNAL)
- no-connect marks 7 -> 25
Other:
- moved on the sheet: U0

Commit message: PCB start
Parts:
- added R1: 120k, Resistor_SMD:R_0201_0603Metric, symbol Device:R_US
- B0: renamed from U0; footprint (none) -> Connector:NS-Tech_Grove_1x04_P2mm_Vertical
- B1: renamed from U1; footprint (none) -> Connector:NS-Tech_Grove_1x04_P2mm_Vertical
- B2: renamed from U2; footprint (none) -> Connector:NS-Tech_Grove_1x04_P2mm_Vertical
- B3: renamed from U3; footprint (none) -> Connector:NS-Tech_Grove_1x04_P2mm_Vertical
Connections:
- net 5V is gone; now on net VCC: A1.27 (+5V), B0.1 (5V), B1.1 (5V), B2.1 (5V), B3.1 (5V), J1.6
- net High: now also R1.1
- net Low: now also R1.2
Other:
- moved on the sheet: B0, B1, B2, B3, J1

Commit message: PCB Draft 1
Parts:
- R1: value 120k -> 120; footprint Resistor_SMD:R_0201_0603Metric -> Resistor_THT:R_Axial_DIN0207_L6.3mm_D2.5mm_P7.62mm_Horizontal
- R3: footprint Resistor_THT:R_Axial_DIN0207_L6.3mm_D2.5mm_P5.08mm_Vertical -> Resistor_THT:R_Axial_DIN0207_L6.3mm_D2.5mm_P7.62mm_Horizontal
Connections:
- net GND is gone; now on net 0: A1.29 (GND), A1.4 (GND), B0.2 (GND), B0.4 (CGND), B1.2 (GND), B1.4 (CGND), B2.2 (GND), B2.4 (CGND), B3.2 (GND), B3.4 (CGND), J1.1
- net High: now also R1.2; no longer R1.1
- net Low: now also R1.1; no longer R1.2
Changed lines of the file:
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@@
 	)
 	(junction
+		(at 250.19 115.57)
+		(diameter 0)
+		(color 0 0 0 0)
+	)
+	(junction
 		(at 144.78 135.89)
 		(diameter 0)
@@
 	)
 	(junction
-		(at 250.19 115.57)
-		(diameter 0)
-		(color 0 0 0 0)
-	)
-	(junction
 		(at 144.78 123.19)
 		(diameter 0)
@@
 	(wire
 		(pts
-			(xy 223.52 144.78) (xy 226.06 144.78)
+			(xy 250.19 115.57) (xy 252.73 115.57)
 		)
 		(stroke
@@
 	(wire
 		(pts
-			(xy 160.02 146.05) (xy 160.02 147.32)
+			(xy 223.52 144.78) (xy 226.06 144.78)
 		)
 		(stroke
@@
 	(wire
 		(pts
-			(xy 156.21 123.19) (xy 144.78 123.19)
+			(xy 160.02 146.05) (xy 160.02 147.32)
 		)
 		(stroke
@@
 	(wire
 		(pts
-			(xy 102.87 85.09) (xy 175.26 85.09)
+			(xy 156.21 123.19) (xy 144.78 123.19)
 		)
 		(stroke
@@
 	(wire
 		(pts
-			(xy 102.87 82.55) (xy 156.21 82.55)
+			(xy 250.19 107.95) (xy 252.73 107.95)
 		)
 		(stroke
@@
 	(wire
 		(pts
-			(xy 250.19 107.95) (xy 252.73 107.95)
+			(xy 102.87 85.09) (xy 175.26 85.09)
 		)
 		(stroke
@@
 	(wire
 		(pts
-			(xy 107.95 62.23) (xy 118.11 62.23)
+			(xy 102.87 82.55) (xy 156.21 82.55)
 		)
 		(stroke
@@
 	(wire
 		(pts
-			(xy 156.21 147.32) (xy 160.02 147.32)
+			(xy 107.95 62.23) (xy 118.11 62.23)
 		)
 		(stroke
@@
 	(wire
 		(pts
-			(xy 175.26 62.23) (xy 193.04 62.23)
+			(xy 156.21 147.32) (xy 160.02 147.32)
 		)
 		(stroke
@@
 	(wire
 		(pts
-			(xy 247.65 107.95) (xy 250.19 107.95)
+			(xy 175.26 62.23) (xy 193.04 62.23)
 		)
 		(stroke
@@
 	(wire
 		(pts
-			(xy 250.19 115.57) (xy 252.73 115.57)
+			(xy 247.65 115.57) (xy 250.19 115.57)
 		)
 		(stroke
@@
 	(wire
 		(pts
-			(xy 247.65 115.57) (xy 250.19 115.57)
-		)
-		(stroke
-			(width 0)
-			(type default)
-		)
-	)
-	(wire
-		(pts
 			(xy 130.81 78.74) (xy 130.81 80.01)
 		)
@@
 	(wire
 		(pts
+			(xy 247.65 107.95) (xy 250.19 107.95)
+		)
+		(stroke
+			(width 0)
+			(type default)
+		)
+	)
+	(wire
+		(pts
 			(xy 156.21 82.55) (xy 156.21 62.23)
 		)
@@
 		)
 	)
+	(global_label "GND"
+		(shape input)
+		(at 201.93 151.13 90)
+		(fields_autoplaced yes)
+		(effects
+			(font
+				(size 1.27 1.27)
+			)
+			(justify left)
+		)
+		(property "Intersheetrefs" "${INTERSHEET_REFS}"
+			(at 201.93 144.2743 90)
+			(hide yes)
+			(show_name no)
+			(do_not_autoplace no)
+			(effects
+				(font
+					(size 1.27 1.27)
+				)
+				(justify left)
+			)
+		)
+	)
 	(global_label "SI"
 		(shape input)
@@
 	)
 	(symbol
+		(lib_id "Simulation_SPICE:0")
+		(at 201.93 151.13 0)
+		(unit 1)
+		(body_style 1)
+		(exclude_from_sim no)
+		(in_bom yes)
+		(on_board yes)
+		(in_pos_files yes)
+		(dnp no)
+		(fields_autoplaced yes)
+		(property "Reference" "#GND02"
+			(at 201.93 156.21 0)
+			(hide yes)
+			(show_name no)
+			(do_not_autoplace no)
+			(effects
+				(font
+					(size 1.27 1.27)
+				)
+			)
+		)
+		(property "Value" "0"
+			(at 201.93 148.59 0)
+			(hide yes)
+			(show_name no)
+			(do_not_autoplace no)
+			(effects
+				(font
+					(size 1.27 1.27)
+				)
+			)
+		)
+		(property "Footprint" ""
+			(at 201.93 151.13 0)
+			(hide yes)
+			(show_name no)
+			(do_not_autoplace no)
+			(effects
+				(font
+					(size 1.27 1.27)
+				)
+			)
+		)
+		(property "Datasheet" "https://ngspice.sourceforge.io/docs/ngspice-html-manual/manual.xhtml#subsec_Circuit_elements__device"
+			(at 201.93 161.29 0)
+			(hide yes)
+			(show_name no)
+			(do_not_autoplace no)
+			(effects
+				(font
+					(size 1.27 1.27)
+				)
+			)
+		)
+		(property "Description" "0V reference potential for simulation"
+			(at 201.93 158.75 0)
+			(hide yes)
+			(show_name no)
+			(do_not_autoplace no)
+			(effects
+				(font
+					(size 1.27 1.27)
+				)
+			)
+		)
+		(pin "1"
+		)
+		(instances
+			(project "Displacement Sensor 2"
+				(path "/cef208de-ab75-42af-9ed7-91863f7f236f"
+					(reference "#GND02")
+					(unit 1)
+				)
+			)
+		)
+	)
+	(symbol
 		(lib_id "Displacement Pins:Displacement_pins")
 		(at 118.11 59.69 0)
@@
 	)
 	(symbol
+		(lib_id "Device:R_US")
+		(at 250.19 111.76 180)
+		(unit 1)
+		(body_style 1)
+		(exclude_from_sim no)
+		(in_bom yes)
+		(on_board yes)
+		(in_pos_files yes)
+		(dnp no)
+		(fields_autoplaced yes)
+		(property "Reference" "R1"
+			(at 252.73 110.4899 0)
+			(show_name no)
+			(do_not_autoplace no)
+			(effects
+				(font
+					(size 1.27 1.27)
+				)
+				(justify right)
+			)
+		)
+		(property "Value" "120"
+			(at 252.73 113.0299 0)
+			(show_name no)
+			(do_not_autoplace no)
+			(effects
+				(font
+					(size 1.27 1.27)
+				)
+				(justify right)
+			)
+		)
+		(property "Footprint" "Resistor_THT:R_Axial_DIN0207_L6.3mm_D2.5mm_P7.62mm_Horizontal"
+			(at 249.174 111.506 90)
+			(hide yes)
+			(show_name no)
+			(do_not_autoplace no)
+			(effects
+				(font
+					(size 1.27 1.27)
+				)
+			)
+		)
+		(property "Datasheet" ""
+			(at 250.19 111.76 0)
+			(hide yes)
+			(show_name no)
+			(do_not_autoplace no)
+			(effects
+				(font
+					(size 1.27 1.27)
+				)
+			)
+		)
+		(property "Description" "Resistor, US symbol"
+			(at 250.19 111.76 0)
+			(hide yes)
+			(show_name no)
+			(do_not_autoplace no)
+			(effects
+				(font
+					(size 1.27 1.27)
+				)
+			)
+		)
+		(pin "1"
+		)
+		(pin "2"
+		)
+		(instances
+			(project "Displacement Sensor 2"
+				(path "/cef208de-ab75-42af-9ed7-91863f7f236f"
+					(reference "R1")
+					(unit 1)
+				)
+			)
+		)
+	)
+	(symbol
 		(lib_id "CAN Integration-altium-import:VCC_BAR")
 		(at 223.52 142.24 180)
@@
 			)
 		)
-		(property "Footprint" "Resistor_THT:R_Axial_DIN0207_L6.3mm_D2.5mm_P5.08mm_Vertical"
+		(property "Footprint" "Resistor_THT:R_Axial_DIN0207_L6.3mm_D2.5mm_P7.62mm_Horizontal"
 			(at 160.274 122.174 90)
 			(hide yes)
@@
 					(unit 1)
 				)
-			)
-		)
-	)
-	(symbol
-		(lib_id "Device:R_US")
-		(at 250.19 111.76 0)
-		(unit 1)
-		(body_style 1)
-		(exclude_from_sim no)
-		(in_bom yes)
-		(on_board yes)
-		(in_pos_files yes)
-		(dnp no)
-		(property "Reference" "R1"
-			(at 248.92 104.14 0)
-			(show_name no)
-			(do_not_autoplace no)
-			(effects
-				(font
-					(size 1.27 1.27)
-				)
-				(justify left)
-			)
-		)
-		(property "Value" "120k"
-			(at 247.904 106.172 0)
-			(show_name no)
-			(do_not_autoplace no)
-			(effects
-				(font
-					(size 1.27 1.27)
-				)
-				(justify left)
-			)
-		)
-		(property "Footprint" "Resistor_SMD:R_0201_0603Metric"
-			(at 251.206 112.014 90)
-			(hide yes)
-			(show_name no)
-			(do_not_autoplace no)
-			(effects
-				(font
-					(size 1.27 1.27)
-				)
-			)
-		)
-		(property "Datasheet" ""
-			(at 250.19 111.76 0)
-			(hide yes)
-			(show_name no)
-			(do_not_autoplace no)
-			(effects
-				(font
-					(size 1.27 1.27)
-				)
-			)
-		)
-		(property "Description" "Resistor, US symbol"
-			(at 250.19 111.76 0)
-			(hide yes)
-			(show_name no)
-			(do_not_autoplace no)
-			(effects
-				(font
-					(size 1.27 1.27)
-				)
-			)
-		)
-		(pin "2"
-		)
-		(pin "1"
-		)
-		(instances
-			(project "Displacement Sensor 2"
-				(path "/cef208de-ab75-42af-9ed7-91863f7f236f"
-					(reference "R1")
-					(unit 1)
-				)
